Commit message: Creating a rough 3D model of JM with URDF

File: dev_ws/src/description/robot_core.xacro (robot description, xacro)
@@ -1,4 +1,5 @@
 <?xml version="1.0"?>
 <robot xmlns:xacro="http://www.ros.org/wiki/xacro">
+    <xacro:include filename="inertial_macros.xacro"/>
     <material name ="white">
         <color rgba="1 1 1 1"/>
@@ -30,4 +31,14 @@
             <material name="white"/>
         </visual>
+        <collision>
+            <origin xyz="0.15 0 0.075"/>
+            <geometry>
+                <box size="0.3 0.3 0.15"/>
+            </geometry>
+            <material name="white"/>
+        </collision>
+        <xacro:inertial_box mass="0.5"   x="0.3" y="0.3" z="0.15">
+            <origin xyz="0.15 0 0.075"/>
+        </xacro:inertial_box>
     </link>
     <!-- LEFT WHEEL -->
@@ -41,8 +52,17 @@
         <visual>
             <geometry>
-                <cylinder length="0.04" radius="0.05" />/>
+                <cylinder length="0.04" radius="0.05" />
             </geometry>
             <material name="blue"/>
         </visual>
+        <collision>
+            <geometry>
+                <cylinder length="0.04" radius="0.05" />
+            </geometry>
+            <material name="blue"/>
+        </collision>
+        <xacro:inertial_cylinder mass="0.1" length="0.04" radius="0.05">
+            <origin xyz="0 0 0" rpy="0 0 0"/>
+        </xacro:inertial_cylinder>
     </link>
     <!-- RIGHT WHEEL -->
@@ -60,4 +80,13 @@
             <material name="blue"/>
         </visual>
+        <collision>
+            <geometry>
+                <cylinder length="0.04" radius="0.05" />/>
+            </geometry>
+            <material name="blue"/>
+        </collision>
+        <xacro:inertial_cylinder mass="0.1" length="0.04" radius="0.05">
+            <origin xyz="0 0 0" rpy="0 0 0"/>
+        </xacro:inertial_cylinder>
     </link>
     <!-- CASTER WHEEL SWIVER PLATE-->
@@ -75,4 +104,13 @@
             <material name="orange"/>
         </visual>
+        <collision>
+            <geometry>
+                <cylinder length="0.1" radius="0.005" />
+            </geometry>
+            <material name="orange"/>
+        </collision>
+        <xacro:inertial_cylinder mass="0.05" length="0.1" radius="0.005">
+            <origin xyz="0 0 0" rpy="0 0 0"/>
+        </xacro:inertial_cylinder>
     </link>
 <!-- CASTER WHEEL-->
@@ -90,4 +128,13 @@
             <material name="blue"/>
         </visual>
+        <collision>
+            <geometry>
+                <cylinder length="0.04" radius="0.05" />
+            </geometry>
+            <material name="blue"/>
+        </collision>
+        <xacro:inertial_cylinder mass="0.1" length="0.04" radius="0.05">
+            <origin xyz="0 0 0" rpy="0 0 0"/>
+        </xacro:inertial_cylinder>
     </link>
 </robot>
